File: Board/Night_Clock_2.brd (EAGLE design)
At the start: 102.8 x 84.8 mm, 65 parts, among them IC1 MEGA8-P, IC2 DS1307, T1 2N3904, T2 2N3904, T3 2N3904, T4 2N3904

Commit message: Gave components  values
Parts:
- C1: value (none) -> 25 V 2200uF
- G1: value B2430UNI -> CR2032
- Q1: value (none) -> 32 Khz
- R1, R2, R3, R4: value (none) -> 470K
- R10, R11, R12, R5, R6, R7, R8, R9: value (none) -> 220
- R13, R14: value (none) -> 2.2K
